File: smerf8-led/smerf8-led.kicad_sch (KiCad schematic)
At the start: 69 parts, among them J1 Conn_Coaxial_Small, J2 Conn_Coaxial_Small, J3 Conn_Coaxial_Small, J4 Conn_Coaxial_Small, U1 ERF8-ERM8-040-DV

Commit message: board 90% done
Parts:
- added TP1, TP10, TP11, TP12, TP13, TP14, TP15, TP16, TP17, TP18, TP19, TP2, TP20, TP21, TP22, TP23, TP24, TP25, TP26, TP27, TP28, TP29, TP3, TP30, TP31, TP32, TP4, TP5, TP6, TP7, TP8, TP9: TestPoint, cody:TestPoint_Plated_Hole_D1.1mm, symbol Connector:TestPoint
- U1: footprint cody:ERF8-040-EM2 -> Library:ERF8-040-EM2
Connections:
- net sig02: no longer J2.1 (In)
- net sig03: no longer J3.1 (In)
- net sig04: no longer J4.1 (In)
- net sig15: now also J3.1 (In)
- net sig16: now also J4.1 (In)
- net sig17: now also J2.1 (In)
- net at D13.2 (A), R13.1: now also TP13.1
- net at D10.2 (A), R10.1: now also TP10.1
- net at D25.2 (A), R25.1: now also TP25.1
- net at D24.2 (A), R24.1: now also TP24.1
- net at D11.2 (A), R11.1: now also TP11.1
- net at D18.2 (A), R18.1: now also TP18.1
- net at D23.2 (A), R23.1: now also TP23.1
- net at D7.2 (A), R7.1: now also TP7.1
- net at D31.2 (A), R31.1: now also TP31.1
- net at D27.2 (A), R27.1: now also TP27.1
- net at D28.2 (A), R28.1: now also TP28.1
- net at D26.2 (A), R26.1: now also TP26.1
- net at D16.2 (A), R16.1: now also TP16.1
- net at D20.2 (A), R20.1: now also TP20.1
- net at D19.2 (A), R19.1: now also TP19.1
- net at D5.2 (A), R5.1: now also TP5.1
- net at D2.2 (A), R2.1: now also TP2.1
- net at D22.2 (A), R22.1: now also TP22.1
- net at D4.2 (A), R4.1: now also TP4.1
- net at D21.2 (A), R21.1: now also TP21.1
- net at D17.2 (A), R17.1: now also TP17.1
- net at D14.2 (A), R14.1: now also TP14.1
- net at D3.2 (A), R3.1: now also TP3.1
- net at D15.2 (A), R15.1: now also TP15.1
- net at D29.2 (A), R29.1: now also TP29.1
- net at D6.2 (A), R6.1: now also TP6.1
- net at D12.2 (A), R12.1: now also TP12.1
- net at D1.2 (A), R1.1: now also TP1.1
- net at D30.2 (A), R30.1: now also TP30.1
- net at D32.2 (A), R32.1: now also TP32.1
- net at D8.2 (A), R8.1: now also TP8.1
- net at D9.2 (A), R9.1: now also TP9.1
Other:
- moved on the sheet: D1, D10, D11, D12, D13, D14, D15, D16, D17, D18, D19, D2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

Commit message: first draft done!
Parts:
- added GND1, GND2, GND3, GND4: TestPoint, TestPoint:TestPoint_Plated_Hole_D2.0mm, symbol mza:TestPoint
Connections:
- net GND: now also GND1.1, GND2.1, GND3.1, GND4.1
